File: hardware/antidote-audio-board/antidote-audio-board.kicad_sch (KiCad schematic)
At the start: 60 parts, among them J1 Cubie GPIO, J2 Instrument Out, J3 Phones, J4 Instrument In, J5 LED Header, J6 I2C Header, SW1 Footswitch, SW2 Footswitch, U1 ADS1115IDGS, U2 MCP6002-xSN, U3 TAC5112IRGER, U4 LP5907MFX-3.3

Commit message: feat: fix schematic issues & document audio bring up
Connections:
- net Phones Mono: no longer J3.R2
- net Phones Sleeve: now also J3.R2
Other:
- moved on the sheet: J3
Changed lines of the file:
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@@
 	(text "For next rev.:\nUse Clean 5V for op-amps\nTo reduce mains hum"
 		(exclude_from_sim no)
-		(at 24.13 123.952 0)
+		(at -44.45 127.762 0)
 		(effects
 			(font
@@
 	)
 	(junction
+		(at 85.09 147.32)
+		(diameter 0)
+		(color 0 0 0 0)
+	)
+	(junction
 		(at 172.72 50.8)
 		(diameter 0)
@@
 	)
 	(junction
+		(at 85.09 139.7)
+		(diameter 0)
+		(color 0 0 0 0)
+	)
+	(junction
 		(at 181.61 212.09)
 		(diameter 0)
@@
 	)
 	(junction
-		(at 74.93 144.78)
-		(diameter 0)
-		(color 0 0 0 0)
-	)
-	(junction
 		(at 66.04 40.64)
 		(diameter 0)
@@
 	)
 	(junction
-		(at 74.93 142.24)
-		(diameter 0)
-		(color 0 0 0 0)
-	)
-	(junction
 		(at 167.64 207.01)
 		(diameter 0)
@@
 	(wire
 		(pts
-			(xy 74.93 137.16) (xy 81.28 137.16)
+			(xy 82.55 139.7) (xy 85.09 139.7)
 		)
 		(stroke
@@
 	(wire
 		(pts
+			(xy 82.55 142.24) (xy 85.09 142.24)
+		)
+		(stroke
+			(width 0)
+			(type default)
+		)
+	)
+	(wire
+		(pts
 			(xy 210.82 90.17) (xy 214.63 90.17)
 		)
@@
 	(wire
 		(pts
-			(xy 74.93 144.78) (xy 81.28 144.78)
+			(xy 85.09 147.32) (xy 90.17 147.32)
 		)
 		(stroke
@@
 	(wire
 		(pts
+			(xy 82.55 144.78) (xy 85.09 144.78)
+		)
+		(stroke
+			(width 0)
+			(type default)
+		)
+	)
+	(wire
+		(pts
 			(xy 25.4 134.62) (xy 25.4 138.43)
 		)
@@
 	(wire
 		(pts
+			(xy 85.09 139.7) (xy 90.17 139.7)
+		)
+		(stroke
+			(width 0)
+			(type default)
+		)
+	)
+	(wire
+		(pts
+			(xy 85.09 142.24) (xy 85.09 139.7)
+		)
+		(stroke
+			(width 0)
+			(type default)
+		)
+	)
+	(wire
+		(pts
 			(xy 115.57 55.88) (xy 119.38 55.88)
 		)
@@
 	(wire
 		(pts
-			(xy 74.93 142.24) (xy 74.93 144.78)
+			(xy 85.09 144.78) (xy 85.09 147.32)
 		)
 		(stroke
@@
 	(wire
 		(pts
-			(xy 74.93 139.7) (xy 74.93 142.24)
+			(xy 82.55 147.32) (xy 85.09 147.32)
 		)
 		(stroke
@@
 	)
 	(label "Phones Sleeve"
-		(at 81.28 137.16 0)
+		(at 90.17 139.7 0)
 		(effects
 			(font
@@
 	)
 	(label "Phones Mono"
-		(at 81.28 144.78 0)
+		(at 90.17 147.32 0)
 		(effects
 			(font
@@
 	(symbol
 		(lib_id "Connector_Audio:AudioJack4")
-		(at 69.85 139.7 0)
+		(at 77.47 142.24 0)
 		(unit 1)
 		(body_style 1)
@@
 		(fields_autoplaced yes)
 		(property "Reference" "J3"
-			(at 67.31 130.81 0)
+			(at 74.93 133.35 0)
 			(show_name no)
 			(do_not_autoplace no)
@@
 		)
 		(property "Value" "Phones"
-			(at 67.31 133.35 0)
+			(at 74.93 135.89 0)
 			(show_name no)
 			(do_not_autoplace no)
@@
 		)
 		(property "Footprint" "Connector_Audio:Jack_3.5mm_PJ320E_Horizontal"
-			(at 69.85 139.7 0)
+			(at 77.47 142.24 0)
 			(hide yes)
 			(show_name no)
@@
 		)
 		(property "Datasheet" ""
-			(at 69.85 139.7 0)
+			(at 77.47 142.24 0)
 			(hide yes)
 			(show_name no)
@@
 		)
 		(property "Description" "Audio Jack, 4 Poles (TRRS)"
-			(at 69.85 139.7 0)
+			(at 77.47 142.24 0)
 			(hide yes)
 			(show_name no)

Commit message: feat: add rc tap to clean op-amp noise
Parts:
- added C21: 10 uF, Capacitor_SMD:C_0603_1608Metric, symbol Device:C
- added R16: 10 K, Resistor_SMD:R_0805_2012Metric, symbol Device:R
Connections:
- net +5V: now also C21.2, R16.1; no longer C13.1, C4.1, R2.1, R7.1
- net GND: now also C21.1
- new net +5V Filtered: C13.1, C4.1, R16.2, R2.1, R7.1
Other:
- moved on the sheet: J3
